Commit message: Update Rizon4s_Grav.urdf
Delet mimic part for the gripper to avoid error in OpenSai simulation.

File: urdf_models/Rizon4s_Grav.urdf (robot description, URDF)
Before this commit: robot rizon4s, 23 links, 22 joints
Links:
- removed link unused_finger_width_link
- link closed_fingers_tcp: mass 0 -> 1E-4
- link grav_tcp: mass 0 -> 1E-4
- link left_finger_tcp: mass 0 -> 1E-4
- link left_finger_tip: mass 0 -> 1E-4
- link right_finger_tcp: mass 0 -> 1E-4
- link right_finger_tip: mass 0 -> 1E-4
Joints:
- removed joint finger_width_joint
- joint closed_fingers_tcp_joint: axis 0 0 1 -> (none)
- joint left_finger_tcp_joint: axis 0 0 1 -> (none)
- joint left_inner_finger_joint: axis 1 0 0 -> (none); limit lower=-0.7854 upper=0.155 effort=0 velocity=2.0 -> (none); mimic joint=left_outer_knuckle_joint multiplier=-1 offset=0 -> (none); origin xyz=0 0 0.058 rpy=0 0 0 -> xyz=0 0 0.058 rpy=0.155 0 0; type revolute -> fixed
- joint left_inner_finger_pad_joint: axis 0 0 1 -> (none)
- joint left_inner_knuckle_joint: axis 1 0 0 -> (none); limit lower=-0.155 upper=0.7854 effort=0 velocity=2.0 -> (none); mimic joint=left_outer_knuckle_joint multiplier=1 offset=0 -> (none); origin xyz=0 -0.0165 0.0995 rpy=0 0 0 -> xyz=0 -0.0165 0.0995 rpy=-0.155 0 0; type revolute -> fixed
- joint left_outer_knuckle_joint: axis 1 0 0 -> (none); limit lower=-0.155 upper=0.7854 effort=0 velocity=2.0 -> (none); mimic joint=finger_width_joint multiplier=9.404 offset=-0.155 -> (none); origin xyz=0 -0.0325 0.0825 rpy=0 0 0 -> xyz=0 -0.0325 0.0825 rpy=-0.155 0 0; type revolute -> fixed
- joint open_fingers_tcp_joint: axis 0 0 1 -> (none)
- joint right_finger_tcp_joint: axis 0 0 1 -> (none)
- joint right_inner_finger_joint: axis 1 0 0 -> (none); limit lower=-0.7854 upper=0.155 effort=0 velocity=2.0 -> (none); mimic joint=left_outer_knuckle_joint multiplier=-1 offset=0 -> (none); origin xyz=0 0 0.058 rpy=0 0 0 -> xyz=0 0 0.058 rpy=0.155 0 0; type revolute -> fixed
- joint right_inner_finger_pad_joint: axis 0 0 1 -> (none)
- joint right_inner_knuckle_joint: axis 1 0 0 -> (none); limit lower=-0.155 upper=0.7854 effort=0 velocity=2.0 -> (none); mimic joint=left_outer_knuckle_joint multiplier=1 offset=0 -> (none); origin xyz=0 0.0165 0.0995 rpy=0 0 3.141592653589793 -> xyz=0 0.0165 0.0995 rpy=-0.155 0 3.141592653589793; type revolute -> fixed
- joint right_outer_knuckle_joint: axis 1 0 0 -> (none); limit lower=-0.155 upper=0.7854 effort=0 velocity=2.0 -> (none); mimic joint=left_outer_knuckle_joint multiplier=1 offset=0 -> (none); origin xyz=0 0.0325 0.0825 rpy=0 0 3.141592653589793 -> xyz=0 0.0325 0.0825 rpy=-0.155 0 3.141592653589793; type revolute -> fixed
